Commit message: default value for transparency parameter

File: colored_link.urdf.xacro (robot description, xacro)
@@ -19,5 +19,5 @@
 -->
 <robot xmlns:xacro="http://www.ros.org/wiki/xacro">
-    <xacro:macro name="colored_link" params="name **visual color transparency **other">
+    <xacro:macro name="colored_link" params="name **visual color transparency:=0 **other">
         <link name="${name}">
             <visual>
